File: lab4/Exercise 2 lab 6/Exercise 2 lab 6.kicad_sch (KiCad schematic)
At the start: 10 parts, among them J1 Conn_01x02_Male, U1 NE555D

Commit message: lab 6
Parts:
- C1: value C_Polarized -> 10μF; footprint (none) -> Capacitor_Tantalum_SMD:CP_EIA-3216-18_Kemet-A_Pad1.58x1.35mm_HandSolder
- C2: value C -> 0.01μF; footprint (none) -> Capacitor_SMD:C_0805_2012Metric_Pad1.18x1.45mm_HandSolder
- D1, D2: footprint (none) -> LED_SMD:LED_1206_3216Metric_Pad1.42x1.75mm_HandSolder
- J1: footprint (none) -> TerminalBlock:TerminalBlock_bornier-2_P5.08mm
- R1, R3, R4: value R -> 1k; footprint (none) -> Resistor_SMD:R_0805_2012Metric_Pad1.20x1.40mm_HandSolder
- R2: value R -> 10k; footprint (none) -> Resistor_SMD:R_0805_2012Metric_Pad1.20x1.40mm_HandSolder
- U1: footprint Package_SO:SOIC-8_3.9x4.9mm_P1.27mm -> Package_SO:SOIC-8-1EP_3.9x4.9mm_P1.27mm_EP2.29x3mm
Connections:
- net +9V: now also J1.1 (Pin_1), R1.1, U1.8 (VCC)
- net GND: now also J1.2 (Pin_2), U1.1 (GND)
- net pin_2: now also C1.1, R2.2
- net pin_7: now also R1.2, R2.1
Other:
- moved on the sheet: C1
