File: lab4/Exercise 2 lab 6/Exercise 2 lab 6.kicad_pcb (KiCad board)
At the start: 2 copper layers, 83.8 x 81.3 mm, 10 parts, among them J1 Conn_01x02_Male, U1 NE555D

Commit message: lab 6
Changed lines of the file:
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@@
   (gr_circle (center 83.82 119.38) (end 83.82 116.84) (layer "Edge.Cuts") (width 0.1) (fill none))
   (gr_rect (start 76.2 48.26) (end 160.02 129.54) (layer "Edge.Cuts") (width 0.1) (fill none))
-  (gr_circle (center 152.4 121.92) (end 155.992102 121.92) (layer "Edge.Cuts") (width 0.1) (fill none))
+  (gr_circle (center 152.4 121.92) (end 154.94 124.46) (layer "Edge.Cuts") (width 0.1) (fill none))
   (gr_circle (center 152.4 55.88) (end 152.4 58.42) (layer "Edge.Cuts") (width 0.1) (fill none))
   (gr_text "EE201 Lab 6" (at 93.98 127) (layer "Edge.Cuts")

Commit message: Gerber Files
Routing:
- net /pin_2: track 85.1 -> 82.5 mm
- net /pin_7: track 61.7 -> 60.8 mm
Other:
- board text added: "EE201 LAB 6"
- board text removed: "EE201 Lab 6"
